Commit message: feat: add wheel

File: my_pkg/description/robot.urdf.xacro (robot description, xacro)
@@ -44,3 +44,27 @@
         <origin xyz="0 0 0" rpy="0 0 0"/>
     </joint>
+    <link name="wheel_left">
+        <visual>
+            <origin xyz="0 0 0" rpy="0 0 0"/>
+            <geometry>
+                <cylinder length="0.05" radius="0.05"/>
+            </geometry>
+            <material name="black"/>
+        </visual>
+        <collision>
+            <origin xyz="0 0 0" rpy="0 0 0"/>
+            <geometry>
+                <cylinder length="0.05" radius="0.05"/>
+            </geometry>
+        </collision>
+        <xacro:inertial_cylinder mass="0.1" length="0.05" radius="0.05">
+            <origin xyz="0 0 0" rpy="0 0 0"/>
+        </xacro:inertial_cylinder>
+    </link>
+    <joint name="chassis_to_wheel_left" type="fixed">
+        <parent link="base_link"/>
+        <child link="wheel_left"/>
+        <origin xyz="0 ${chassis_width/2 + 0.03} ${0.05/2}" rpy="1.57 0 0"/>
+        <axis xyz="0 0 1"/>
+    </joint>
 </robot>

Commit message: feat: urdf improve

File: my_pkg/description/robot.urdf.xacro (robot description, xacro)
@@ -62,6 +62,6 @@
         </xacro:inertial_cylinder>
     </link>
-    <joint name="chassis_to_wheel_left" type="fixed">
-        <parent link="base_link"/>
+    <joint name="chassis_to_wheel_left" type="continuous">
+        <parent link="chassis"/>
         <child link="wheel_left"/>
         <origin xyz="0 ${chassis_width/2 + 0.03} ${0.05/2}" rpy="1.57 0 0"/>

Commit message: feat: right wheel

File: my_pkg/description/robot.urdf.xacro (robot description, xacro)
@@ -68,3 +68,27 @@
         <axis xyz="0 0 1"/>
     </joint>
+    <link name="wheel_right">
+        <visual>
+            <origin xyz="0 0 0" rpy="0 0 0"/>
+            <geometry>
+                <cylinder length="0.05" radius="0.05"/>
+            </geometry>
+            <material name="black"/>
+        </visual>
+        <collision>
+            <origin xyz="0 0 0" rpy="0 0 0"/>
+            <geometry>
+                <cylinder length="0.05" radius="0.05"/>
+            </geometry>
+        </collision>
+        <xacro:inertial_cylinder mass="0.1" length="0.05" radius="0.05">
+            <origin xyz="0 0 0" rpy="0 0 0"/>
+        </xacro:inertial_cylinder>
+    </link>
+    <joint name="chassis_to_wheel_right" type="continuous">
+        <parent link="chassis"/>
+        <child link="wheel_right"/>
+        <origin xyz="0 -${chassis_width/2 + 0.03} ${0.05/2}" rpy="1.57 0 0"/>
+        <axis xyz="0 0 1"/>
+    </joint>
 </robot>
