Commit message: feat: detect obstacle

File: my_pkg/description/lidar.xacro (robot description, xacro)
@@ -4,5 +4,5 @@
         <parent link="chassis"/>
         <child link="laser_frame"/>
-        <origin xyz="0.122 0 0.212" rpy="0 0 0"/>
+        <origin xyz="0.122 0 0.180" rpy="0 0 0"/>
     </joint>
     <link name="laser_frame">
@@ -41,6 +41,6 @@
                   <samples>640</samples>
                   <resolution>1</resolution>
-                  <min_angle>-1.396263</min_angle>
-                  <max_angle>1.396263</max_angle>
+                  <min_angle>-1.57</min_angle>
+                  <max_angle>1.57</max_angle>
                 </horizontal>
                 <vertical>
@@ -53,5 +53,5 @@
               <range>
                 <min>0.08</min>
-                <max>10.0</max>
+                <max>15.0</max>
                 <resolution>0.01</resolution>
               </range>

File: my_pkg/description/robot.urdf.xacro (robot description, xacro)
@@ -5,4 +5,11 @@
     <xacro:property name="chassis_width" value="0.2"/>
     <xacro:property name="chassis_height" value="0.1"/>
+    <xacro:property name="wheel_offset_x" value="0.226"/>
+    <xacro:property name="wheel_offset_y" value="0.1485"/>
+    <xacro:property name="wheel_offset_z" value="0.01"/>
+    <xacro:property name="caster_wheel_radius" value="0.03"/>
+    <xacro:property name="caster_wheel_mass" value="0.01"/>
+    <xacro:property name="caster_wheel_offset_x" value="0.20"/>
+    <xacro:property name="caster_wheel_offset_z" value="-0.010"/>
     <material name="white">
         <color rgba="1 1 1 1" />
@@ -92,3 +99,25 @@
         <axis xyz="0 0 1"/>
     </joint>
+    <!-- CASTER WHEEL LINK -->
+    <joint name="caster_wheel_joint" type="fixed">
+        <parent link="chassis"/>
+        <child link="caster_wheel"/>
+        <origin xyz="${caster_wheel_offset_x} 0 ${caster_wheel_offset_z}"/>
+    </joint>
+    <link name="caster_wheel">
+        <visual>
+            <geometry>
+                <sphere radius="${caster_wheel_radius}"/>
+            </geometry>
+            <material name="white"/>
+        </visual>
+        <collision>
+            <geometry>
+                <sphere radius="${caster_wheel_radius}"/>
+            </geometry>
+        </collision>
+        <xacro:inertial_sphere mass="${caster_wheel_mass}" radius="${caster_wheel_radius}">
+            <origin xyz="0 0 0" rpy="0 0 0"/>
+        </xacro:inertial_sphere>
+    </link>
 </robot>
