Commit message: fix: add caster

File: my_pkg/description/gazebo_control.xacro (robot description, xacro)
@@ -5,6 +5,6 @@
             <left_joint>chassis_to_wheel_left</left_joint>
             <right_joint>chassis_to_wheel_right</right_joint>
-            <wheel_separation>0.297</wheel_separation>
-            <wheel_radius>0.033</wheel_radius>
+            <wheel_separation>0.20</wheel_separation>
+            <wheel_radius>0.05</wheel_radius>
             <topic>cmd_vel</topic>
             <max_linear_acceleration>0.33</max_linear_acceleration>

File: my_pkg/description/robot.urdf.xacro (robot description, xacro)
@@ -5,11 +5,13 @@
     <xacro:property name="chassis_width" value="0.2"/>
     <xacro:property name="chassis_height" value="0.1"/>
+    <xacro:property name="chassis_mass" value="1.0"/>
     <xacro:property name="wheel_offset_x" value="0.226"/>
     <xacro:property name="wheel_offset_y" value="0.1485"/>
     <xacro:property name="wheel_offset_z" value="0.01"/>
+    <xacro:property name="wheel_mass" value="0.5"/>
     <xacro:property name="caster_wheel_radius" value="0.03"/>
-    <xacro:property name="caster_wheel_mass" value="0.01"/>
-    <xacro:property name="caster_wheel_offset_x" value="0.20"/>
-    <xacro:property name="caster_wheel_offset_z" value="-0.010"/>
+    <xacro:property name="caster_wheel_mass" value="0.05"/>
+    <xacro:property name="caster_wheel_offset_x" value="0.26"/>
+    <xacro:property name="caster_wheel_offset_z" value="0.006"/>
     <material name="white">
         <color rgba="1 1 1 1" />
@@ -41,5 +43,5 @@
             </geometry>
         </collision>
-        <xacro:inertial_box mass="0.5" x="${chassis_length}" y="${chassis_width}" z="${chassis_height}">
+        <xacro:inertial_box mass="${chassis_mass}" x="${chassis_length}" y="${chassis_width}" z="${chassis_height}">
             <origin xyz="${chassis_length/2} 0 ${chassis_height/2}" rpy="0 0 0"/>
         </xacro:inertial_box>
@@ -65,5 +67,5 @@
             </geometry>
         </collision>
-        <xacro:inertial_cylinder mass="0.1" length="0.05" radius="0.05">
+        <xacro:inertial_cylinder mass="${wheel_mass}" length="0.05" radius="0.05">
             <origin xyz="0 0 0" rpy="0 0 0"/>
         </xacro:inertial_cylinder>
@@ -89,5 +91,5 @@
             </geometry>
         </collision>
-        <xacro:inertial_cylinder mass="0.1" length="0.05" radius="0.05">
+        <xacro:inertial_cylinder mass="${wheel_mass}" length="0.05" radius="0.05">
             <origin xyz="0 0 0" rpy="0 0 0"/>
         </xacro:inertial_cylinder>
